File: pcb/pcb.sch (KiCad schematic (older format))
At the start: 14 parts

Commit message: added first switch
Parts:
- added D?: D_Small, symbol Device:D_Small
- added MX?: MX-NoLED, symbol MX_Alps_Hybrid:MX-NoLED
Changed lines of the file:
@@
 Wire Wire Line
 	8250 4150 8450 4150
+$Comp
+L MX_Alps_Hybrid:MX-NoLED MX?
+U 1 1 61836743
+P 1150 1800
+F 0 "MX?" H 1183 2023 60  0000 C CNN
+F 1 "MX-NoLED" H 1183 1949 20  0000 C CNN
+F 2 "" H 525 1775 60  0001 C CNN
+F 3 "" H 525 1775 60  0001 C CNN
+	1    1150 1800
+	1    0    0    -1
+$EndComp
+$Comp
+L Device:D_Small D?
+U 1 1 61837541
+P 1100 2050
+F 0 "D?" V 1146 1980 50  0000 R CNN
+F 1 "D_Small" V 1055 1980 50  0000 R CNN
+F 2 "" V 1100 2050 50  0001 C CNN
+F 3 "~" V 1100 2050 50  0001 C CNN
+	1    1100 2050
+	0    -1   -1   0
+$EndComp
 $EndSCHEMATC

Commit message: added basic keyboard matrix
Parts:
- added D? (x86): D_Small, symbol Device:D_Small
- added MX? (x86): MX-NoLED, symbol MX_Alps_Hybrid:MX-NoLED
Other:
- moved on the sheet: C?, R?, SW?, U?, Y?
